Commit message: update gazebo

File: src/robot_fablab/urdf/robot_fablab.xacro (robot description, xacro)
@@ -3,4 +3,11 @@
   xmlns:xacro="http://www.ros.org/wiki/xacro">
   <xacro:include filename="$(find robot_fablab)/urdf/robot_fablab.gazebo"/>
+<link name="base_footprint">
+  <visual>
+    <geometry>
+      <box size="0.001 0.001 0.001"/>
+    </geometry>
+  </visual>
+</link>
   <joint name="base_footprint_joint" type="fixed">
     <parent link="base_footprint"/>

Commit message: update

File: src/robot_fablab/urdf/robot_fablab.xacro (robot description, xacro)
@@ -3,11 +3,11 @@
   xmlns:xacro="http://www.ros.org/wiki/xacro">
   <xacro:include filename="$(find robot_fablab)/urdf/robot_fablab.gazebo"/>
-<link name="base_footprint">
-  <visual>
-    <geometry>
-      <box size="0.001 0.001 0.001"/>
-    </geometry>
-  </visual>
-</link>
+  <link name="base_footprint">
+    <visual>
+      <geometry>
+        <box size="0.001 0.001 0.001"/>
+      </geometry>
+    </visual>
+  </link>
   <joint name="base_footprint_joint" type="fixed">
     <parent link="base_footprint"/>
